Commit message: changed the asset and limits

File: assets/urdf/hexapod.urdf (robot description, URDF)
Before this commit: robot pexod, 25 links, 24 joints
Joints:
- joint body_leg_0: limit lower=-2.0944 upper=2.0944 effort=1.961 velocity=5.236 -> lower=-0.3491 upper=0.3491 effort=1.961 velocity=5.236
- joint body_leg_1: limit lower=-2.0944 upper=2.0944 effort=1.961 velocity=5.236 -> lower=-0.3491 upper=0.3491 effort=1.961 velocity=5.236
- joint body_leg_2: limit lower=-2.0944 upper=2.0944 effort=1.961 velocity=5.236 -> lower=-0.3491 upper=0.3491 effort=1.961 velocity=5.236
- joint body_leg_3: limit lower=-2.0944 upper=2.0944 effort=1.961 velocity=5.236 -> lower=-0.3491 upper=0.3491 effort=1.961 velocity=5.236
- joint body_leg_4: limit lower=-2.0944 upper=2.0944 effort=1.961 velocity=5.236 -> lower=-0.3491 upper=0.3491 effort=1.961 velocity=5.236
- joint body_leg_5: limit lower=-2.0944 upper=2.0944 effort=1.961 velocity=5.236 -> lower=-0.3491 upper=0.3491 effort=1.961 velocity=5.236
- joint leg_0_1_2: limit lower=-2.0944 upper=2.0944 effort=1.961 velocity=5.236 -> lower=-0.3491 upper=0.3491 effort=1.961 velocity=5.236
- joint leg_0_2_3: limit lower=-2.0944 upper=2.0944 effort=1.961 velocity=5.236 -> lower=-0.3491 upper=0.3491 effort=1.961 velocity=5.236
- joint leg_1_1_2: limit lower=-2.0944 upper=2.0944 effort=1.961 velocity=5.236 -> lower=-0.3491 upper=0.3491 effort=1.961 velocity=5.236
- joint leg_1_2_3: limit lower=-2.0944 upper=2.0944 effort=1.961 velocity=5.236 -> lower=-0.3491 upper=0.3491 effort=1.961 velocity=5.236
- joint leg_2_1_2: limit lower=-2.0944 upper=2.0944 effort=1.961 velocity=5.236 -> lower=-0.3491 upper=0.3491 effort=1.961 velocity=5.236
- joint leg_2_2_3: limit lower=-2.0944 upper=2.0944 effort=1.961 velocity=5.236 -> lower=-0.3491 upper=0.3491 effort=1.961 velocity=5.236
- joint leg_3_1_2: limit lower=-2.0944 upper=2.0944 effort=1.961 velocity=5.236 -> lower=-0.3491 upper=0.3491 effort=1.961 velocity=5.236
- joint leg_3_2_3: limit lower=-2.0944 upper=2.0944 effort=1.961 velocity=5.236 -> lower=-0.3491 upper=0.3491 effort=1.961 velocity=5.236
- joint leg_4_1_2: limit lower=-2.0944 upper=2.0944 effort=1.961 velocity=5.236 -> lower=-0.3491 upper=0.3491 effort=1.961 velocity=5.236
- joint leg_4_2_3: limit lower=-2.0944 upper=2.0944 effort=1.961 velocity=5.236 -> lower=-0.3491 upper=0.3491 effort=1.961 velocity=5.236
- joint leg_5_1_2: limit lower=-2.0944 upper=2.0944 effort=1.961 velocity=5.236 -> lower=-0.3491 upper=0.3491 effort=1.961 velocity=5.236
- joint leg_5_2_3: limit lower=-2.0944 upper=2.0944 effort=1.961 velocity=5.236 -> lower=-0.3491 upper=0.3491 effort=1.961 velocity=5.236
